Commit message: Fixed nav2 transform tolerance and urdf tweaks for Lidar alignment

File: src/gastrobot_bringup/urdf/gastrobot.urdf (robot description, URDF)
Before this commit: robot gastrobot, 5 links, 4 joints
Links:
- added link left_wheel; visual cylinder length=0.04 radius=0.072
- added link right_wheel; visual cylinder length=0.04 radius=0.072
- link tower_link: geometry visual box size=0.2 0.2 0.66
Joints:
- added joint left_wheel_joint: type fixed, parent base_link, child left_wheel, origin xyz=0 0.24 -0.024 rpy=0 0 0
- added joint right_wheel_joint: type fixed, parent base_link, child right_wheel, origin xyz=0 -0.24 -0.024 rpy=0 0 0
- joint base_joint: origin xyz=0 0 0.08 rpy=0 0 0 -> xyz=0 0 0.096 rpy=0 0 0
- joint laser_joint: origin xyz=0 0 0.66 rpy=0 0 0 -> xyz=0 0 0.66 rpy=0 0 3.14159
- joint tower_joint: origin xyz=-0.145 0 0.31 rpy=0 0 0 -> xyz=-0.15 0 0.31 rpy=0 0 0

Commit message: STABLE BASELINE: fixed LiDAR TF orientation, stable SLAM, heading hold implemented, drivetrain + odometry validated

File: src/gastrobot_bringup/urdf/gastrobot.urdf (robot description, URDF)
Before this commit: robot gastrobot, 13 links, 12 joints
Joints:
- joint tower_joint: origin xyz=-0.15 0 0.31 rpy=0 0 0 -> xyz=-0.0 0 0.31 rpy=0 0 0
